File: RelayBoard_V2/relay.brd (EAGLE design)
At the start: 157.5 x 57.1 mm, 30 parts, among them K1 T9AS1D12-5, K2 T9AS1D12-5, T1 2N2222, T2 2N2222, T3 2N2222, T4 2N2222, X1 22-23-2021

Commit message: change power receptacles to thru hole
Parts:
- removed U$12: PIN_5X2_SOCKET, BloomWall:PIN_5X2_SOCKET
- removed U$13, U$14, U$15: MAIN, BloomWall:MAIN
- added U$4: 9POS_MINI_DIN, BloomWall:9POS_MINI_DIN
- added U$5: IEC_MALE, BloomWall:IEC_MALE
- added U$6, U$7: IEC_FEMALE, BloomWall:IEC_FEMALE
- U$1: value PIN_20X2 -> PIN_20X2_NOTFLIPPED; device BloomWall:PIN_20X2 -> BloomWall:PIN_20X2_NOTFLIPPED
- moved U$1 136.5 mm to (-90.2, -111.8)
- moved OK2 45.8 mm to (52.1, 19.1)
- moved T2 18.3 mm to (24.1, 38.1)
- moved K1 12.7 mm to (17.8, 11.4)
Connections:
- removed net 3.3V2: U$1.3.3V2
- removed net GND8: U$1.GND8
- removed net N$42: U$12.P$1, U$9.PGND
- new net 3_3V: U$1.3_3V
- new net 3_3V1: U$1.3_3V1
- new net 5V: U$1.5V
- new net 5V1: U$1.5V1
- new net GND2: U$1.GND2
- new net GND3: U$1.GND3
- new net GND4: U$1.GND4
- new net N$31: U$4.P9, U$9.PGND
- net DGND: now also U$1.GPIO12, U$4.P8; no longer U$1.GND, U$12.P$9
- net N$1: now also U$1.ID_SC; no longer U$1.GPIO27
- net N$17: now also U$7.HOT; no longer U$15.HOT
- net N$19: now also U$5.HOT; no longer U$13.HOT
- net N$2: now also U$1.GND1; no longer U$1.GPIO17
- net N$20: now also U$5.NEUTRAL, U$6.NEUTRAL, U$7.NEUTRAL; no longer U$13.NEUTRAL, U$14.NEUTRAL, U$15.NEUTRAL
- net N$21: now also U$1.GPIO6; no longer U$1.GPIO15
- net N$28: now also U$1.GND6; no longer U$1.GPIO23
- net N$29: now also U$1.SCLK; no longer U$1.GPIO24
- net N$30: now also U$1.GPIO19; no longer U$1.GND4
- net N$33: now also U$1.GPIO26; no longer U$1.5V2
- net N$34: now also U$1.GPIO17; no longer U$1.GND7
- net N$35: now also U$1.GND, U$4.P5; no longer U$1.GPIO4, U$12.P$8
- net N$36: now also U$1.GPIO21, U$4.P4; no longer U$1.3.3V, U$12.P$7
- net N$37: now also U$4.P7; no longer U$12.P$6
- net N$38: no longer U$12.P$5
- net N$39: no longer U$12.P$4
- net N$40: no longer U$12.P$3
- net N$41: now also U$4.P6; no longer U$12.P$2
- net N$6: now also U$1.GND7; no longer U$1.5V
- net N$7: now also U$1.GPIO13; no longer U$1.GPIO14
- net N$9: now also U$6.HOT; no longer U$14.HOT
- net PGND: now also U$5.GND, U$6.GROUND, U$7.GROUND; no longer U$13.GROUND, U$14.GROUND, U$15.GROUND
Other:
- board size 157.5 x 57.1 mm -> 157.5 x 85 mm
