File: PCB/FreshBytes.sch (EAGLE design)
At the start: 30 parts, among them K1 T9AS1D12-5, K2 T9AS1D12-5, T1 2N2222, T2 2N2222, T3 2N2222, T4 2N2222, X1 22-23-2021

Commit message: Swap to R Pi Zero W as the brains
Power inlet may be in the wrong location. Will commit again tomorrow with proper spot.
Parts:
- removed K1, K2: T9AS1D12-5, BloomWall:T9AS1D12-5
- added U$11: RELAY, FreshBytes:RELAY
- added U$13: RPI_ZERO, FreshBytes:RPI_ZERO
- U$1: value PIN_20X2_NOTFLIPPED -> POWER_IN; device BloomWall:PIN_20X2_NOTFLIPPED -> FreshBytes:POWER_IN
- U$12: value MAIN -> RELAY; device BloomWall:MAIN -> FreshBytes:RELAY
Connections:
- net DGND: now also U$13.GPIO12; no longer U$1.GPIO12
- net GND: now also U$13.GND, U$13.GND1, U$13.GND2, U$13.GND3, U$13.GND4, U$13.GND5, U$13.GND6, U$13.GND7; no longer U$1.GND, U$1.GND1, U$1.GND2, U$1.GND3, U$1.GND4, U$1.GND5, U$1.GND6, U$1.GND7
- net N$1: now also U$13.ID_SC; no longer U$1.ID_SC
- net N$16: now also U$12.COIL2; no longer K2.COIL2
- net N$17: now also U$12.NO; no longer K2.NO
- net N$18: now also U$11.COIL2; no longer K1.COIL2
- net N$19: now also U$1.HOT, U$11.COM, U$12.COM; no longer K1.COM, K2.COM, U$12.HOT
- net N$20: now also U$1.NEUTRAL; no longer U$12.NEUTRAL
- net N$21: now also U$13.GPIO6; no longer U$1.GPIO6
- net N$29: now also U$13.SCLK; no longer U$1.SCLK
- net N$30: now also U$13.GPIO19; no longer U$1.GPIO19
- net N$32: now also U$11.COIL1, U$12.COIL1; no longer K1.COIL1, K2.COIL1
- net N$33: now also U$13.GPIO26; no longer U$1.GPIO26
- net N$34: now also U$13.GPIO17; no longer U$1.GPIO17
- net N$36: now also U$13.GPIO21; no longer U$1.GPIO21
- net N$38: now also U$4.P3
- net N$39: now also U$4.P1
- net N$40: now also U$4.P2
- net N$7: now also U$13.GPIO13; no longer U$1.GPIO13
- net N$9: now also U$11.NO; no longer K1.NO
- net PGND: now also U$1.GND; no longer U$12.GROUND
Other:
- moved on the sheet: R9

Commit message: Fix drill size for RPi headers. Swapping over to Rhino for CAD stuff
Parts:
- removed U$13: RPI_ZERO, FreshBytes:RPI_ZERO
- added U$10: RPI_ZERO, FreshBytes:RPI_ZERO
Connections:
- removed net N$30: MUX.GND, MUX.INH, MUX.VEE, U$13.GPIO19, U$5.GND, U$8.GND, U$9.GND
- removed net N$34: R7.2, R8.2, U$13.GPIO17
- new net N$35: R1.2, U$10.GPIO17
- new net N$42: R9.1, U$10.GPIO4, U$4.P5
- new net N$43: MUX.B, R8.1, U$10.GPIO23
- new net N$44: R3.2, R4.2, U$10.5V
- net DGND: now also U$10.GND; no longer U$13.GPIO12
- net GND: now also MUX.GND, MUX.INH, MUX.VEE, R7.2, R8.2, U$10.GND2, U$10.GND3, U$10.GND4, U$10.GND7, U$10.GND8, U$5.GND, U$8.GND, U$9.GND; no longer MUX.B, R1.2, R3.2, R4.2, R8.1, R9.1, U$13.GND, U$13.GND1, U$13.GND2, U$13.GND3, U$13.GND4, U$13.GND5, U$13.GND6, U$13.GND7, U$4.P5
- net N$1: now also U$10.GPIO27; no longer U$13.ID_SC
- net N$21: now also U$10.RX; no longer U$13.GPIO6
- net N$29: now also U$10.GPIO24; no longer U$13.SCLK
- net N$33: now also U$10.5V2; no longer U$13.GPIO26
- net N$36: now also U$10.3.3V; no longer U$13.GPIO21
- net N$7: now also U$10.TX; no longer U$13.GPIO13
